Commit message: Add reward and state to bipedal env

File: gym/urdf/robot.urdf (robot description, URDF)
Before this commit: robot bipedal, 7 links, 6 joints
Joints:
- joint core_left_hip: limit lower=0.0 upper=3.14159 effort=1000.0 velocity=0.5 -> lower=-0.785398 upper=0.785398 effort=1000.0 velocity=0.5
- joint core_right_hip: limit lower=0.0 upper=3.14159 effort=1000.0 velocity=0.5 -> lower=0.785398 upper=0.785398 effort=1000.0 velocity=0.5
